File: KiCAD-project-files/LED-dimmer.kicad_pcb (KiCad board)
At the start: 2 copper layers, 41.9 x 25.4 mm, 12 parts, among them IC1 ATTINY85-S, P1 CONN_01X02, P2 CONN_01X02, P3 CONN_02X03, Q1 Q_NMOS_GDSD, U1 AP1117D50

Commit message: Added PDF
Parts:
- renumbered IC1 to U1, U1 to U2
Other:
- board text added: "+12V"
- board text added: "+5v"
- board text added: "GND"
- board text added: "LED-GND"
- board text added: "gnd"
Changed lines of the file:
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@@
     (links 26)
     (no_connects 0)
-    (area 176.310219 115.97088 222.9702 143.585001)
+    (area 177.089999 118.034999 219.150001 143.585001)
     (thickness 1.6)
-    (drawings 14)
+    (drawings 19)
     (tracks 133)
     (zones 0)
@@
     (pad_to_mask_clearance 0.2)
     (aux_axis_origin 0 0)
-    (visible_elements FFFFFF7F)
+    (visible_elements FFFFFFFF)
     (pcbplotparams
       (layerselection 0x010f0_80000001)
-      (usegerberextensions false)
+      (usegerberextensions true)
       (excludeedgelayer true)
       (linewidth 0.100000)
@@
     (descr "Potentiometer, Wire Pads only, RevA, 30 July 2010,")
     (tags "Potentiometer, Wire Pads only, RevA, 30 July 2010,")
-    (fp_text reference RV1 (at 0.0508 -3.49758 180) (layer F.SilkS)
-      (effects (font (size 1 1) (thickness 0.15)))
-    )
-    (fp_text value POT (at -1.34874 13.25118 180) (layer F.Fab)
+    (fp_text reference RV1 (at 2.286 7.92226 180) (layer F.SilkS) hide
+      (effects (font (size 1 1) (thickness 0.15)))
+    )
+    (fp_text value POT (at 3.048 4.93776 270) (layer F.Fab)
       (effects (font (size 1 1) (thickness 0.15)))
     )
@@
     (tags "CMS SOJ")
     (attr smd)
-    (fp_text reference IC1 (at 0 -1.27 270) (layer F.SilkS)
+    (fp_text reference U1 (at 3.302 0 360) (layer F.SilkS)
       (effects (font (size 1 1) (thickness 0.15)))
     )
@@
     (tags "capacitor 0805")
     (attr smd)
-    (fp_text reference C2 (at 0 -2.1 180) (layer F.SilkS)
+    (fp_text reference C2 (at -3.429 0 180) (layer F.SilkS)
       (effects (font (size 1 1) (thickness 0.15)))
     )
@@
     (at 215.392 133.604 270)
     (descr "2-way 5mm pitch terminal block, Phoenix MKDS series")
-    (fp_text reference P1 (at 2.5 5.9 270) (layer F.SilkS)
+    (fp_text reference P1 (at 2.5 5.842 270) (layer F.SilkS) hide
       (effects (font (size 1 1) (thickness 0.15)))
     )
@@
     (at 215.392 123.19 270)
     (descr "2-way 5mm pitch terminal block, Phoenix MKDS series")
-    (fp_text reference P2 (at 2.5 5.9 270) (layer F.SilkS)
+    (fp_text reference P2 (at 2.5 5.588 270) (layer F.SilkS) hide
       (effects (font (size 1 1) (thickness 0.15)))
     )
@@
     (descr "Through hole pin header")
     (tags "pin header")
-    (fp_text reference P3 (at 0 -5.1 180) (layer F.SilkS)
+    (fp_text reference P3 (at -2.54 2.413 270) (layer F.SilkS) hide
       (effects (font (size 1 1) (thickness 0.15)))
     )
@@
     (tags "resistor 0603")
     (attr smd)
-    (fp_text reference R1 (at 0 -1.9 270) (layer F.SilkS)
-      (effects (font (size 1 1) (thickness 0.15)))
-    )
-    (fp_text value 1k (at 0 1.9 270) (layer F.Fab)
+    (fp_text reference R1 (at 0 1.4605 450) (layer F.SilkS)
+      (effects (font (size 1 1) (thickness 0.15)))
+    )
+    (fp_text value 1k (at 0.3175 2.0955 270) (layer F.Fab)
       (effects (font (size 1 1) (thickness 0.15)))
     )
@@
     (tags "resistor 0603")
     (attr smd)
-    (fp_text reference R2 (at 0 -1.9 180) (layer F.SilkS)
+    (fp_text reference R2 (at -3.175 0 180) (layer F.SilkS)
       (effects (font (size 1 1) (thickness 0.15)))
     )
@@
     (tags "D-Pak TO252AA Diode")
     (attr smd)
-    (fp_text reference Q1 (at 0 -7.5 90) (layer F.SilkS)
+    (fp_text reference Q1 (at 4.572 4.318 180) (layer F.SilkS)
       (effects (font (size 1 1) (thickness 0.15)))
     )
@@
     (tags "CMS SOT")
     (attr smd)
-    (fp_text reference U1 (at 0 -0.762 270) (layer F.SilkS)
+    (fp_text reference U2 (at -4.191 3.302 360) (layer F.SilkS)
       (effects (font (size 1 1) (thickness 0.15)))
     )
@@
     (descr "module 1 pin (ou trou mecanique de percage)")
     (tags DEV)
-    (fp_text reference REF** (at 0 -3.048) (layer F.SilkS)
+    (fp_text reference REF** (at 0 -3.048) (layer F.SilkS) hide
       (effects (font (size 1 1) (thickness 0.15)))
     )
@@
     (pad 1 thru_hole circle (at 0 0) (size 3.2 3.2) (drill 3.2) (layers *.Cu *.Mask F.SilkS))
   )
+  (gr_text LED-GND (at 213.233 142.367) (layer F.SilkS)
+    (effects (font (size 1.5 1.5) (thickness 0.3)))
+  )
+  (gr_text GND (at 215.392 119.507) (layer F.SilkS)
+    (effects (font (size 1.5 1.5) (thickness 0.3)))
+  )
+  (gr_text +12V (at 209.55 130.937 90) (layer F.SilkS)
+    (effects (font (size 1.5 1.5) (thickness 0.3)))
+  )
+  (gr_text gnd (at 181.483 130.302) (layer B.SilkS)
+    (effects (font (size 1.5 1.5) (thickness 0.3)) (justify left mirror))
+  )
+  (gr_text +5v (at 181.61 120.269) (layer B.SilkS)
+    (effects (font (size 1.3 1.3) (thickness 0.3)) (justify left mirror))
+  )
   (gr_line (start 177.165 118.11) (end 183.515 118.11) (layer Edge.Cuts) (width 0.15))
