File: KiCAD-project-files/LED-dimmer.sch (KiCad schematic (older format))
At the start: 11 parts, among them IC1 ATTINY85-S, P1 CONN_01X02, P2 CONN_01X02, P3 CONN_02X03, Q1 Q_NMOS_GDSD, U1 AP1117D50

Commit message: Added PDF
Parts:
- renumbered IC1 to U1, U1 to U2
Connections:
- net +12V: now also P1.1 (P1); no longer P1.2 (P2)
- net at Q1.4 (D): now also P1.2 (P2); no longer P1.1 (P1)
Changed lines of the file:
@@
 $EndDescr
 $Comp
-L ATTINY85-S IC1
+L ATTINY85-S U1
 U 1 1 5675C516
 P 5400 2400
-F 0 "IC1" H 4250 2800 50  0000 C CNN
+F 0 "U1" H 4250 2800 50  0000 C CNN
 F 1 "ATTINY85-S" H 6400 2000 50  0000 C CNN
 F 2 "SMD_Packages:SOIC-8-N" H 6350 2400 50  0000 C CIN
@@
 F 3 "" H 2600 2250 50  0000 C CNN
 	1    2600 2250
-	-1   0    0    1
+	-1   0    0    -1
 $EndComp
 $Comp
@@
 	2850 2300 2850 2350
 $Comp
-L AP1117D50 U1
+L AP1117D50 U2
 U 1 1 567604B5
 P 5550 950
-F 0 "U1" H 5650 700 50  0000 C CNN
+F 0 "U2" H 5650 700 50  0000 C CNN
 F 1 "AP1117D50" H 5550 1200 50  0000 C CNN
 F 2 "TO_SOT_Packages_SMD:SOT-223" H 5550 950 50  0001 C CNN
